File: board/MCTheremin.sch (KiCad schematic (older format))
At the start: 92 parts, among them J1 Barrel_Jack, J10 Conn_01x02, J11 Conn_01x01, J12 Conn_01x01, J13 Conn_01x01, J14 Conn_01x01, J15 Conn_01x01, J16 Conn_01x01, J17 Conn_01x02, J18 Conn_01x01, J19 Conn_01x04, J2 Conn_01x02, J20 Conn_01x04, J21 Conn_01x02, J22 Conn_01x02, J3 Conn_01x01, J4 Conn_01x01, J5 Conn_01x02, J6 Conn_01x02, J7 Conn_01x01, J8 Conn_01x01, J9 Conn_01x01, Q1 2N3904, Q2 2N3904, Q3 2N3904, SW1 SW_Push, SW2 SW_Push, U1 74HC04, U2 MCP4921, U3 LM7805_TO220, U4 LM386, U5 LM358, U6 74HC04

Commit message: Pre LC
Parts:
- added R25: 1k, Resistors_THT:R_Axial_DIN0207_L6.3mm_D2.5mm_P7.62mm_Horizontal, symbol R
- R10: value 10k -> 220R
Connections:
- net at U5.6 (-), U5.7: now also R25.1; no longer C13.1
- new net: C13.1, R25.2
Other:
- moved on the sheet: C13, J17, R10
Changed lines of the file:
@@
 L CP C13
 U 1 1 5B5303FF
-P 5650 5150
-F 0 "C13" H 5675 5250 50  0000 L CNN
-F 1 "220 uF" H 5675 5050 50  0000 L CNN
-F 2 "Capacitors_THT:CP_Radial_D7.5mm_P2.50mm" H 5688 5000 50  0001 C CNN
-F 3 "" H 5650 5150 50  0001 C CNN
-	1    5650 5150
+P 6050 5550
+F 0 "C13" H 6075 5650 50  0000 L CNN
+F 1 "220 uF" H 6075 5450 50  0000 L CNN
+F 2 "Capacitors_THT:CP_Radial_D7.5mm_P2.50mm" H 6088 5400 50  0001 C CNN
+F 3 "" H 6050 5550 50  0001 C CNN
+	1    6050 5550
 	0    -1   -1   0
 $EndComp
@@
 L R R10
 U 1 1 5B530CAF
-P 5900 5300
-F 0 "R10" V 5980 5300 50  0000 C CNN
-F 1 "10k" V 5900 5300 50  0000 C CNN
-F 2 "Resistors_THT:R_Axial_DIN0207_L6.3mm_D2.5mm_P7.62mm_Horizontal" V 5830 5300 50  0001 C CNN
-F 3 "" H 5900 5300 50  0001 C CNN
-	1    5900 5300
+P 6300 5700
+F 0 "R10" V 6380 5700 50  0000 C CNN
+F 1 "220R" V 6300 5700 50  0000 C CNN
+F 2 "Resistors_THT:R_Axial_DIN0207_L6.3mm_D2.5mm_P7.62mm_Horizontal" V 6230 5700 50  0001 C CNN
+F 3 "" H 6300 5700 50  0001 C CNN
+	1    6300 5700
 	1    0    0    -1
 $EndComp
@@
 L Conn_01x02 J17
 U 1 1 5B530D85
-P 6300 5150
-F 0 "J17" H 6300 5250 50  0000 C CNN
-F 1 "Conn_01x02" H 6300 4950 50  0000 C CNN
-F 2 "Connectors_Terminal_Blocks:TerminalBlock_bornier-2_P5.08mm" H 6300 5150 50  0001 C CNN
-F 3 "" H 6300 5150 50  0001 C CNN
-	1    6300 5150
+P 6700 5550
+F 0 "J17" H 6700 5650 50  0000 C CNN
+F 1 "Conn_01x02" H 6700 5350 50  0000 C CNN
+F 2 "Connectors_Terminal_Blocks:TerminalBlock_bornier-2_P5.08mm" H 6700 5550 50  0001 C CNN
+F 3 "" H 6700 5550 50  0001 C CNN
+	1    6700 5550
 	1    0    0    -1
 $EndComp
@@
 L GND #PWR46
 U 1 1 5B53121E
-P 5900 5550
-F 0 "#PWR46" H 5900 5300 50  0001 C CNN
-F 1 "GND" H 5900 5400 50  0000 C CNN
-F 2 "" H 5900 5550 50  0001 C CNN
-F 3 "" H 5900 5550 50  0001 C CNN
-	1    5900 5550
+P 6300 5950
+F 0 "#PWR46" H 6300 5700 50  0001 C CNN
+F 1 "GND" H 6300 5800 50  0000 C CNN
+F 2 "" H 6300 5950 50  0001 C CNN
+F 3 "" H 6300 5950 50  0001 C CNN
+	1    6300 5950
 	1    0    0    -1
 $EndComp
@@
 L GND #PWR47
 U 1 1 5B53153C
-P 6050 5450
-F 0 "#PWR47" H 6050 5200 50  0001 C CNN
-F 1 "GND" H 6050 5300 50  0000 C CNN
-F 2 "" H 6050 5450 50  0001 C CNN
-F 3 "" H 6050 5450 50  0001 C CNN
-	1    6050 5450
+P 6450 5850
+F 0 "#PWR47" H 6450 5600 50  0001 C CNN
+F 1 "GND" H 6450 5700 50  0000 C CNN
+F 2 "" H 6450 5850 50  0001 C CNN
+F 3 "" H 6450 5850 50  0001 C CNN
+	1    6450 5850
 	1    0    0    -1
 $EndComp
@@
 	4400 6450 4400 6500
 Wire Wire Line
-	5800 5150 6100 5150
-Connection ~ 5900 5150
-Wire Wire Line
-	5350 5150 5500 5150
-Wire Wire Line
-	5900 5450 5900 5550
-Wire Wire Line
-	6050 5450 6050 5250
-Wire Wire Line
-	6050 5250 6100 5250
+	6200 5550 6500 5550
+Connection ~ 6300 5550
+Wire Wire Line
+	5350 5150 5650 5150
+Wire Wire Line
+	6300 5850 6300 5950
+Wire Wire Line
+	6450 5850 6450 5650
+Wire Wire Line
+	6450 5650 6500 5650
 Wire Wire Line
 	6850 950  6850 1050
@@
 	2900 5700 2700 5700
 Wire Wire Line
-	2700 5400 2400 5400
+	2400 5400 2700 5400
 Wire Wire Line
 	2500 6000 2500 5700
@@
 Text Notes 7350 6950 0    60   ~ 0
 MC Theremin by Daniel Marks\nSeptember 15, 2018 version
+$Comp
+L R R25
+U 1 1 5B9E7551
+P 5650 5300
+F 0 "R25" V 5730 5300 50  0000 C CNN
+F 1 "1k" V 5650 5300 50  0000 C CNN
+F 2 "Resistors_THT:R_Axial_DIN0207_L6.3mm_D2.5mm_P7.62mm_Horizontal" V 5580 5300 50  0001 C CNN
+F 3 "" H 5650 5300 50  0001 C CNN
+	1    5650 5300
+	1    0    0    -1
+$EndComp
+Wire Wire Line
+	5650 5450 5650 5550
+Wire Wire Line
+	5650 5550 5900 5550
 $EndSCHEMATC

Commit message: Changed to LC oscillator - removed copper fill from under oscillator
Parts:
- added C23, C24: 100 pF, Capacitors_THT:C_Disc_D5.0mm_W2.5mm_P5.00mm, symbol C
- added C25, C26: 220 pF, Capacitors_THT:C_Disc_D5.0mm_W2.5mm_P5.00mm, symbol C
- added L1, L2: 1 mH, Inductors_THT:L_Axial_L7.0mm_D3.3mm_P12.70mm_Horizontal_Fastron_MICC, symbol L
- C8: value 33 pF -> 100 pF
- C9: value 47 pF -> 100 pF
- R1, R2: value 10k -> 2.2M
- R7, R8: value 10k -> 220R
Connections:
- net GND: now also U6.11, U6.13, U6.9, C23.2, C24.2, C25.1, C26.1; no longer U6.1, U6.3, U6.5
- net at U1.10, U1.9: no longer C9.1
- net at U1.11, U1.12: now also R2.1, R7.1
- net at R1.1: now also R8.1, U6.2, U6.3; no longer U6.13
- net at C8.2, J5.1 (Pin_1), J5.2 (Pin_2)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: now also L1.2; no longer R1.2, R7.2
- net at R22.1, U1.8: no longer R8.1
- net at U1.13: now also C9.1, R2.2, C24.1; no longer R2.1
- net at C9.2, J6.1 (Pin_1), J6.2 (Pin_2)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: now also L2.2; no longer R2.2, R8.2
- net at U6.12: no longer U6.11
- net at U6.4: now also U6.5
- net at U6.6: now also R20.1
- new net: C23.1, C8.1, R1.2, U6.1
- new net: C25.2, L1.1, R8.2
- new net: C26.2, L2.1, R7.2
- now unconnected: U6.10, U6.8
- no-connect marks 10 -> 9
Other:
- moved on the sheet: J5, J6, J7, J8, U1D, U1E, U1F, U6A, U6B, U6C, U6D, U6E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

Commit message: First working MCTheremin with LC oscillators
Parts:
- C23: value 100 pF -> 150 pF
- C24: value 100 pF -> 220 pF
- C25: value 220 pF -> 150 pF
- L1, L2: value 1 mH -> 400 uH
- R7, R8: value 220R -> 1k
Changed lines of the file:
@@
 P 1550 1100
 F 0 "C23" H 1575 1200 50  0000 L CNN
-F 1 "100 pF" H 1575 1000 50  0000 L CNN
+F 1 "150 pF" H 1575 1000 50  0000 L CNN
 F 2 "Capacitors_THT:C_Disc_D5.0mm_W2.5mm_P5.00mm" H 1588 950 50  0001 C CNN
 F 3 "" H 1550 1100 50  0001 C CNN
@@
 P 2950 1500
 F 0 "R8" V 3030 1500 50  0000 C CNN
-F 1 "220R" V 2950 1500 50  0000 C CNN
+F 1 "1k" V 2950 1500 50  0000 C CNN
 F 2 "Resistors_THT:R_Axial_DIN0207_L6.3mm_D2.5mm_P7.62mm_Horizontal" V 2880 1500 50  0001 C CNN
 F 3 "" H 2950 1500 50  0001 C CNN
@@
 P 2900 2900
 F 0 "R7" V 2980 2900 50  0000 C CNN
-F 1 "220R" V 2900 2900 50  0000 C CNN
+F 1 "1k" V 2900 2900 50  0000 C CNN
 F 2 "Resistors_THT:R_Axial_DIN0207_L6.3mm_D2.5mm_P7.62mm_Horizontal" V 2830 2900 50  0001 C CNN
 F 3 "" H 2900 2900 50  0001 C CNN
@@
 P 2350 1750
 F 0 "L1" V 2300 1750 50  0000 C CNN
-F 1 "1 mH" V 2425 1750 50  0000 C CNN
+F 1 "400 uH" V 2425 1750 50  0000 C CNN
 F 2 "Inductors_THT:L_Axial_L7.0mm_D3.3mm_P12.70mm_Horizontal_Fastron_MICC" H 2350 1750 50  0001 C CNN
 F 3 "" H 2350 1750 50  0001 C CNN
@@
 P 2400 3100
 F 0 "L2" V 2350 3100 50  0000 C CNN
-F 1 "1 mH" V 2475 3100 50  0000 C CNN
+F 1 "400 uH" V 2475 3100 50  0000 C CNN
 F 2 "Inductors_THT:L_Axial_L7.0mm_D3.3mm_P12.70mm_Horizontal_Fastron_MICC" H 2400 3100 50  0001 C CNN
 F 3 "" H 2400 3100 50  0001 C CNN
@@
 P 1550 2500
 F 0 "C24" H 1575 2600 50  0000 L CNN
-F 1 "100 pF" H 1575 2400 50  0000 L CNN
+F 1 "220 pF" H 1575 2400 50  0000 L CNN
 F 2 "Capacitors_THT:C_Disc_D5.0mm_W2.5mm_P5.00mm" H 1588 2350 50  0001 C CNN
 F 3 "" H 1550 2500 50  0001 C CNN
@@
 P 3250 1500
 F 0 "C25" H 3275 1600 50  0000 L CNN
-F 1 "220 pF" H 3275 1400 50  0000 L CNN
+F 1 "150 pF" H 3275 1400 50  0000 L CNN
 F 2 "Capacitors_THT:C_Disc_D5.0mm_W2.5mm_P5.00mm" H 3288 1350 50  0001 C CNN
 F 3 "" H 3250 1500 50  0001 C CNN

Commit message: Accidental connection in LM358
Parts:
- R25: value 1k -> 220R
Connections:
- net at C6.1, R24.2, R4.2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: no longer U5.1, U5.2 (-), U5.5 (+)
- new net: U5.1, U5.2 (-), U5.5 (+)
Changed lines of the file:
@@
 P 5650 5300
 F 0 "R25" V 5730 5300 50  0000 C CNN
-F 1 "1k" V 5650 5300 50  0000 C CNN
+F 1 "220R" V 5650 5300 50  0000 C CNN
 F 2 "Resistors_THT:R_Axial_DIN0207_L6.3mm_D2.5mm_P7.62mm_Horizontal" V 5580 5300 50  0001 C CNN
 F 3 "" H 5650 5300 50  0001 C CNN
@@
 Wire Wire Line
 	9950 3600 10200 3600
-Connection ~ 3750 5050
 Wire Wire Line
 	2550 5050 3800 5050
@@
 	4400 6150 4400 6100
 Connection ~ 4500 5150
-Connection ~ 4650 5050
-Wire Wire Line
-	3750 4800 4650 4800
-Wire Wire Line
-	3750 5050 3750 4800
-Wire Wire Line
-	4650 4800 4650 5150
+Wire Wire Line
+	4650 5150 4650 5050
 Wire Wire Line
 	4750 5050 4650 5050
@@
 	4000 4750 4000 4850
 Wire Wire Line
-	4650 5150 4400 5150
+	4400 5150 4650 5150
 Wire Wire Line
 	4500 5600 4500 5150
@@
 	2200 1300 1850 1300
 Wire Wire Line
-	1850 1300 1850 850
+	1850 850  1850 1300
 Wire Wire Line
 	1400 850  1950 850
